File: Schematics/SolarScavenger/SolarScavenger.kicad_pcb (KiCad board)
At the start: 2 copper layers, 38 parts, among them J1 SolarConnector, J10 CH1_OUT, J11 CH2_OUT, J12 CH3_OUT, J13 CH4_OUT, J2 PROGRAMMING, J3 BatteryPack, J4 ESC_PWM_CONTROL, J5 ESC_connector, J6 CH1_IN, J7 CH2_IN, J8 CH3_IN, J9 CH4_IN, Q1 IRLML2502, Q2 IRLML2502, U1 4N25, U2 AP1117-33, U3 ESP32-WROOM-E, U4 INA219AxD

Commit message: PCB final candidate
Parts:
- removed J9: CH4_IN, Connector_PinHeader_2.54mm:PinHeader_1x03_P2.54mm_Vertical
- added G***: LOGO, GluonLib:LogoGluon_12mm, F.Cu at (141.7, 68.6)
- added J14: CH1_OUT, Connector_PinHeader_2.54mm:PinHeader_1x03_P2.54mm_Vertical, F.Cu at (172.5, 39.4)
- added J15: CH2_OUT, Connector_PinHeader_2.54mm:PinHeader_1x03_P2.54mm_Vertical, F.Cu at (172.5, 41.9)
- added J16: CH3_OUT, Connector_PinHeader_2.54mm:PinHeader_1x03_P2.54mm_Vertical, F.Cu at (172.5, 44.5)
- added J17: CH4_OUT, Connector_PinHeader_2.54mm:PinHeader_1x03_P2.54mm_Vertical, F.Cu at (172.5, 47.0)
- added JP6: INA_A0, Jumper:SolderJumper-2_P1.3mm_Open_Pad1.0x1.5mm, F.Cu at (147.1, 75.4)
- added JP7: INA_A1, Jumper:SolderJumper-2_P1.3mm_Open_Pad1.0x1.5mm, F.Cu at (143.9, 75.4)
- added R13: 1k, Resistor_SMD:R_1206_3216Metric_Pad1.30x1.75mm_HandSolder, F.Cu at (132.8, 81.3)
- added R14: 1k, Resistor_SMD:R_1206_3216Metric_Pad1.30x1.75mm_HandSolder, F.Cu at (143.4, 79.7)
- added R15: 330, Resistor_SMD:R_1206_3216Metric_Pad1.30x1.75mm_HandSolder, F.Cu at (148.4, 79.7)
- added R16: 1k, Resistor_SMD:R_1206_3216Metric_Pad1.30x1.75mm_HandSolder, F.Cu at (131.4, 73.4)
- added R17: 1k, Resistor_SMD:R_1206_3216Metric_Pad1.30x1.75mm_HandSolder, F.Cu at (131.4, 76.5)
- added R18: R100/2W, Resistor_SMD:R_2512_6332Metric_Pad1.40x3.35mm_HandSolder, F.Cu at (139.2, 91.1)
- added R19: R100/2W, Resistor_SMD:R_2512_6332Metric_Pad1.40x3.35mm_HandSolder, F.Cu at (139.2, 86.1)
- added R20: 47k, Resistor_SMD:R_1206_3216Metric_Pad1.30x1.75mm_HandSolder, F.Cu at (124.2, 53.7)
- added REF**: MountingHole_3.2mm_M3_Pad, MountingHole:MountingHole_3.2mm_M3_Pad, F.Cu at (105.0, 53.3)
- added REF**: MountingHole_3.2mm_M3_Pad, MountingHole:MountingHole_3.2mm_M3_Pad, F.Cu at (175.0, 53.3)
- added REF**: MountingHole_3.2mm_M3_Pad, MountingHole:MountingHole_3.2mm_M3_Pad, F.Cu at (123.0, 88.0)
- added REF**: MountingHole_3.2mm_M3_Pad, MountingHole:MountingHole_3.2mm_M3_Pad, F.Cu at (157.0, 88.0)
- added U5: INA219AxD, Package_SO:SOIC-8_3.9x4.9mm_P1.27mm, F.Cu at (137.3, 79.1)
- added kibuzzard-63EE93D3: G***, kibuzzard-63EE93D3, F.Cu at (168.1, 66.5)
- added kibuzzard-63EE93FE: G***, kibuzzard-63EE93FE, F.Cu at (168.1, 64.0)
- added kibuzzard-63EE93FE: G***, kibuzzard-63EE93FE, F.Cu at (168.1, 41.9)
- added kibuzzard-63EE940D: G***, kibuzzard-63EE940D, F.Cu at (168.1, 39.4)
- added kibuzzard-63EE941D: G***, kibuzzard-63EE941D, F.Cu at (168.1, 61.5)
- added kibuzzard-63EE9442: G***, kibuzzard-63EE9442, F.Cu at (168.1, 44.5)
- added kibuzzard-63EE9448: G***, kibuzzard-63EE9448, F.Cu at (168.1, 58.9)
- added kibuzzard-63EE9448: G***, kibuzzard-63EE9448, F.Cu at (168.1, 47.0)
- added kibuzzard-63F118E7: G***, kibuzzard-63F118E7, F.Cu at (175.0, 36.3)
- added kibuzzard-63F118F7: G***, kibuzzard-63F118F7, F.Cu at (175.0, 69.6)
- D1, D2: footprint LED_THT:LED_D5.0mm -> LED_SMD:LED_1210_3225Metric_Pad1.42x2.65mm_HandSolder
- J10: value CH1_OUT -> CH1_IN
- J11: value CH2_OUT -> CH2_IN
- J12: value CH3_OUT -> CH3_IN
- J13: value CH4_OUT -> CH4_IN
- J6: value CH1_IN -> Micro_SD_Card; footprint Connector_PinHeader_2.54mm:PinHeader_1x03_P2.54mm_Vertical -> microSD:microSD-Receptacle-SelfEject
- J7: value CH2_IN -> RUDDER_POT
- J8: value CH3_IN -> THROTTLE_POt
- R1: value 220 -> 300
- R10, R9: value 1k -> 47k; footprint Resistor_SMD:R_1020_2550Metric_Pad1.33x5.20mm_HandSolder -> Resistor_SMD:R_1206_3216Metric_Pad1.30x1.75mm_HandSolder
- R11, R12: value R100/2W -> 47k; footprint Resistor_SMD:R_2512_6332Metric_Pad1.40x3.35mm_HandSolder -> Resistor_SMD:R_1206_3216Metric_Pad1.30x1.75mm_HandSolder
- R3: value 300 -> 220
- R4: value 1k -> 4k7
- R5: value 10k -> R_Photo; footprint Resistor_SMD:R_1020_2550Metric_Pad1.33x5.20mm_HandSolder -> Connector_PinHeader_2.54mm:PinHeader_1x02_P2.54mm_Vertical
- R6: footprint Resistor_SMD:R_1020_2550Metric_Pad1.33x5.20mm_HandSolder -> Resistor_SMD:R_1206_3216Metric_Pad1.30x1.75mm_HandSolder
- R7: value 1k -> 10k; footprint Resistor_SMD:R_1020_2550Metric_Pad1.33x5.20mm_HandSolder -> Resistor_SMD:R_1206_3216Metric_Pad1.30x1.75mm_HandSolder
- R8: value 330 -> 47k; footprint Resistor_SMD:R_1020_2550Metric_Pad1.33x5.20mm_HandSolder -> Resistor_SMD:R_1206_3216Metric_Pad1.30x1.75mm_HandSolder
- U1: value 4N25 -> DS18B20; footprint Package_DIP:DIP-6_W7.62mm -> Package_TO_SOT_THT:TO-92_Inline
- U2: value AP1117-33 -> 4N25; footprint Package_TO_SOT_SMD:SOT-223-3_TabPin2 -> Package_DIP:DIP-6_W7.62mm
- U3: value ESP32-WROOM-E -> AP1117-33; footprint Espressif:ESP32-WROOM-32E -> Package_TO_SOT_THT:TO-220-3_Vertical
- U4: value INA219AxD -> ESP32-WROOM-E; footprint Package_SO:SOIC-8_3.9x4.9mm_P1.27mm -> Espressif:ESP32-WROOM-32E
- moved J2 81.7 mm to (153.4, 36.6)
- moved J12 78.5 mm to (172.5, 61.5), turned to 90 degrees
- moved J11 73.2 mm to (172.5, 64.0), turned to 90 degrees
- moved J13 62.8 mm to (172.5, 58.9), turned to 90 degrees
- moved R12 54.9 mm to (121.9, 53.7), turned to -90 degrees
- moved U1 54.2 mm to (158.9, 40.4), turned to 90 degrees
- moved R11 52.4 mm to (119.6, 53.7), turned to -90 degrees
- moved R8 52.1 mm to (112.7, 53.7), turned to -90 degrees
- moved JP4 52.0 mm to (161.5, 56.1), turned to 180 degrees
- moved R10 49.5 mm to (117.3, 53.7), turned to -90 degrees
- moved JP2 45.8 mm to (153.9, 56.1), turned to 180 degrees
- moved R5 44.7 mm to (112.0, 61.2)
- moved R7 44.4 mm to (128.3, 41.4), turned to 90 degrees
- moved R9 44.3 mm to (115.0, 53.7), turned to -90 degrees
- moved JP1 44.0 mm to (144.5, 62.5), turned to -90 degrees
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Connections:
- D1 pad 2: Net-(D1-Pad2) -> Net-(D1-A)
- D2 pad 2: Net-(D2-Pad2) -> Net-(D2-A)
- J1 pad 1: SUPPLY_IN_P -> MOTOR_SUPPLY_N
- J1 pad 2: MOTOR_SUPPLY_N -> SUPPLY_IN_P
- J10 pad 1: Net-(J10-Pad1) -> Net-(J10-Pin_1)
- J11 pad 1: Net-(J11-Pad1) -> Net-(J11-Pin_1)
- J12 pad 1: Net-(J12-Pad1) -> Net-(J12-Pin_1)
- J13 pad 1: Net-(J13-Pad1) -> Net-(J13-Pin_1)
- J3 pad 2: Net-(J3-Pad2) -> Net-(J3-Pin_2)
- J5 pad 1: MOTOR_SUPPLY_P -> MOTOR_SUPPLY_N
- J5 pad 2: MOTOR_SUPPLY_N -> MOTOR_SUPPLY_P
- J6 pad 1: Net-(J6-Pad1) -> /SD_DATA2
- J6 pad 2: ESC_5V -> /SD_DATA3
- J6 pad 3: MOTOR_SUPPLY_N -> /SD_CMD
- J7 pad 1: Net-(J7-Pad1) -> MOTOR_SUPPLY_N
- J7 pad 2: ESC_5V -> RUDDER_ADC
- J7 pad 3: MOTOR_SUPPLY_N -> +3V3
- J8 pad 1: Net-(J8-Pad1) -> MOTOR_SUPPLY_N
- J8 pad 2: ESC_5V -> THROTTLE_ADC
- J8 pad 3: MOTOR_SUPPLY_N -> +3V3
- JP2 pad 1: Net-(J6-Pad1) -> Net-(J10-Pin_1)
- JP2 pad 2: Net-(J10-Pad1) -> Net-(J14-Pin_1)
- JP3 pad 1: Net-(J7-Pad1) -> Net-(J11-Pin_1)
- JP3 pad 2: Net-(J11-Pad1) -> Net-(J15-Pin_1)
- JP4 pad 1: Net-(J8-Pad1) -> Net-(J12-Pin_1)
- JP4 pad 2: Net-(J12-Pad1) -> Net-(J16-Pin_1)
- JP5 pad 1: Net-(J9-Pad1) -> Net-(J13-Pin_1)
- JP5 pad 2: Net-(J13-Pad1) -> Net-(J17-Pin_1)
- R1 pad 1: PWM_TO_ESC -> ESC_5V
- R1 pad 2: Net-(R1-Pad2) -> Net-(D1-A)
- R10 pad 1: INA_SCL -> /SD_CMD
- R11 pad 1: SUPPLY_IN_P -> /SD_DATA0
- R11 pad 2: MOTOR_SUPPLY_P -> +3V3
- R12 pad 1: SUPPLY_IN_P -> /SD_DATA1
- R12 pad 2: MOTOR_SUPPLY_P -> +3V3
- R2 pad 2: Net-(D1-Pad2) -> Net-(D2-A)
- R3 pad 1: ESC_5V -> PWM_TO_ESC
- R3 pad 2: Net-(D2-Pad2) -> Net-(R3-Pad2)
- R4 pad 1: ESC_PWM -> +3V3
- R4 pad 2: ESC_GND -> LIGHT_SENSOR
- R5 pad 1: MOTOR_SUPPLY_N -> LIGHT_SENSOR
- R5 pad 2: +3V3 -> MOTOR_SUPPLY_N
- R6 pad 1: Net-(R6-Pad1) -> ESC_PWM
- R6 pad 2: MOTOR_SUPPLY_P -> ESC_GND
- R7 pad 1: MOTOR_VOLTAGE -> MOTOR_SUPPLY_N
- R7 pad 2: Net-(R6-Pad1) -> +3V3
- R8 pad 1: MOTOR_SUPPLY_N -> /SD_DATA2
- R8 pad 2: MOTOR_VOLTAGE -> +3V3
- R9 pad 1: +3V3 -> /SD_DATA3
- R9 pad 2: INA_SDA -> +3V3
- U1 pad 1: Net-(R1-Pad2) -> MOTOR_SUPPLY_N
- U1 pad 2: MOTOR_SUPPLY_N -> TEMP_SENSOR
- U1 pad 3: unconnected-(U1-Pad3) -> +3V3
- U2 pad 1: MOTOR_SUPPLY_N -> Net-(R3-Pad2)
- U2 pad 2: +3V3 -> MOTOR_SUPPLY_N
- U2 pad 3: Net-(J3-Pad2) -> unconnected-(U2-NC-Pad3)
- U3 pad 3: MOTOR_SUPPLY_N -> Net-(J3-Pin_2)
- U4 pad 1: +3V3 -> MOTOR_SUPPLY_N
- U4 pad 3: INA_SDA -> MOTOR_SUPPLY_N
- U4 pad 4: INA_SCL -> MOTOR_VOLTAGE
- U4 pad 5: +3V3 -> LIGHT_SENSOR
- U4 pad 6: MOTOR_SUPPLY_N -> unconnected-(U4-GPIO34/ADC1_CH6-Pad6)
- U4 pad 7: MOTOR_SUPPLY_P -> unconnected-(U4-GPIO35/ADC1_CH7-Pad7)
- U4 pad 8: SUPPLY_IN_P -> TEMP_SENSOR
Routing:
- net MOTOR_SUPPLY_N: track 0.00 -> 135.6 mm, vias 0 -> 1
- net +3V3: track 0.00 -> 123.8 mm
- net MOTOR_VOLTAGE: track 0.00 -> 48.1 mm, vias 0 -> 2
- net ESC_5V: track 0.00 -> 44.0 mm
- net LED_2: track 0.00 -> 41.4 mm, vias 0 -> 2
- net /SD_CMD: track 0.00 -> 35.8 mm, vias 0 -> 2
- net /SD_DATA0: track 0.00 -> 34.4 mm, vias 0 -> 2
- net /SD_DATA1: track 0.00 -> 33.4 mm, vias 0 -> 2
- net LED_1: track 0.00 -> 32.9 mm, vias 0 -> 2
- net TEMP_SENSOR: track 0.00 -> 32.1 mm, vias 0 -> 1
- net /SD_DATA3: track 0.00 -> 29.3 mm, vias 0 -> 2
- net PWM_TO_ESC: track 0.00 -> 27.2 mm, vias 0 -> 2
- net Net-(J14-Pin_1): track 0.00 -> 25.8 mm
- net /SD_DATA2: track 0.00 -> 25.3 mm, vias 0 -> 2
- net /SD_CLK: track 0.00 -> 23.4 mm, vias 0 -> 2
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- added copper zone on B.Cu, net MOTOR_SUPPLY_N
- added copper zone on F.Cu, net MOTOR_SUPPLY_N
Other:
- board outline added: 80 x 63.3 mm
- board text added: "Solar Scavenger v1.0"

Commit message: Actual final canditate
Parts:
- added kibuzzard-63F11AB2: G***, kibuzzard-63F11AB2, F.Cu at (156.6, 39.1)
- added kibuzzard-63F11AB7: G***, kibuzzard-63F11AB7, F.Cu at (156.6, 41.6)
- added kibuzzard-63F11AC7: G***, kibuzzard-63F11AC7, F.Cu at (157.0, 44.2)
- added kibuzzard-63F11AD1: G***, kibuzzard-63F11AD1, F.Cu at (157.0, 36.6)
- added kibuzzard-63F11F4E: G***, kibuzzard-63F11F4E, F.Cu at (139.4, 66.8)
- added kibuzzard-63F11F5A: G***, kibuzzard-63F11F5A, F.Cu at (144.5, 66.0)
- added kibuzzard-63F12006: G***, kibuzzard-63F12006, F.Cu at (110.7, 78.2)
- added kibuzzard-63F12026: G***, kibuzzard-63F12026, F.Cu at (159.6, 71.6)
- added kibuzzard-63F127EF: G***, kibuzzard-63F127EF, F.Cu at (128.5, 67.8)
- added kibuzzard-63F1280A: G***, kibuzzard-63F1280A, F.Cu at (128.5, 65.3)
- added kibuzzard-63F12816: G***, kibuzzard-63F12816, F.Cu at (128.5, 62.7)
- moved U2 36.8 mm to (163.8, 61.0)
- moved J4 30.3 mm to (151.1, 71.6)
- moved R6 30.3 mm to (153.4, 76.5)
- moved R3 27.5 mm to (154.4, 59.4), turned to 0 degrees
- moved G*** 24.8 mm to (119.9, 80.3)
- moved U1 3.44 mm to (161.8, 38.6)
- moved R7 1.27 mm to (127.0, 41.4)
Routing:
- net +3V3: track 123.8 -> 170.2 mm, vias 0 -> 2
- net INA_SCL: track 2.47 -> 48.4 mm, vias 0 -> 2
- net INA_SDA: track 5.95 -> 45.0 mm, vias 0 -> 2
- net LIGHT_SENSOR: track 0.00 -> 38.2 mm, vias 0 -> 2
- net ESC_5V: track 44.0 -> 71.7 mm
- net LED_2: track 41.4 -> 53.9 mm
- net PWM_TO_ESC: track 27.2 -> 14.7 mm
- net LED_1: track 32.9 -> 40.3 mm
- net Net-(R3-Pad2): track 2.29 -> 8.47 mm
- net ESC_PWM: track 9.62 -> 14.0 mm
- net TEMP_SENSOR: track 32.1 -> 35.8 mm
- net MOTOR_SUPPLY_N: track 135.6 -> 138.7 mm, vias 1 -> 7
- net RUDDER_ADC: track 15.2 -> 16.6 mm
- net THROTTLE_ADC: track 19.1 -> 20.3 mm
- net /SD_DATA0: track 34.4 -> 33.8 mm
Other:
- outline, holes or cut-outs redrawn
- board text added: "Solar Scavenger v1.0 @LabGluon @Prediktor"
- board text removed: "Solar Scavenger v1.0"

Commit message: Version 1.0 de la PCB, enviada a fabricar
Parts:
- moved G*** 2.42 mm to (119.8, 77.9)
Routing:
- net MOTOR_SUPPLY_N: vias 7 -> 8
Other:
- board text added: "Gracias a: @spuertes @carlosbetdev @araba_st @kukudrulu @fateuki1 @andygm_ @un_bizco"
Changed lines of the file:
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@@
   )
   (footprint "GluonLib:LogoGluon_12mm" (layer "F.Cu")
-    (at 119.888 80.264)
+    (at 119.761 77.851)
     (attr through_hole)
     (fp_text reference "G***" (at 0 0) (layer "F.SilkS") hide
@@
       (stroke (width 0) (type solid)) (fill solid) (layer "F.SilkS"))
   )
+  (gr_line (start 123.825 67.437) (end 110.871 67.437)
+    (stroke (width 0.15) (type default)) (layer "B.SilkS"))
   (gr_line (start 180 69.492) (end 180 33)
     (stroke (width 0.1) (type default)) (layer "Edge.Cuts"))
@@
   (gr_line (start 130.5 39.5) (end 150 39.5)
     (stroke (width 0.1) (type default)) (layer "Edge.Cuts"))
-  (gr_text "Solar Scavenger v1.0\n@LabGluon\n@Prediktor\n" (at 110.744 74.168) (layer "F.SilkS")
+  (gr_text "Gracias a:\n\n@spuertes\n@carlosbetdev\n@araba_st\n@kukudrulu\n@fateuki1\n@andygm_\n@un_bizco" (at 123.317 79.375) (layer "B.SilkS")
+    (effects (font (size 1 1) (thickness 0.15)) (justify left bottom mirror))
+  )
+  (gr_text "Solar Scavenger v1.0\n@LabGluon\n@Prediktor\n" (at 109.601 71.882) (layer "F.SilkS")
     (effects (font (size 1 1) (thickness 0.15)) (justify left bottom))
   )
@@
   (via (at 136.398 43.688) (size 0.8) (drill 0.4) (layers "F.Cu" "B.Cu") (free) (net 6))
   (via (at 139.954 53.086) (size 0.8) (drill 0.4) (layers "F.Cu" "B.Cu") (free) (net 6))
+  (via (at 153.543 64.389) (size 0.8) (drill 0.4) (layers "F.Cu" "B.Cu") (free) (net 6))
   (segment (start 130 86.066) (end 149.92 86.066) (width 2) (layer "B.Cu") (net 6))
   (segment (start 149.272 86.066) (end 149.352 86.146) (width 2) (layer "B.Cu") (net 6))

Commit message: PCB v1.1
Parts:
- removed G***: LOGO, GluonLib:LogoGluon_12mm
- removed J10: CH1_IN, Connector_PinHeader_2.54mm:PinHeader_1x03_P2.54mm_Vertical
- removed J11: CH2_IN, Connector_PinHeader_2.54mm:PinHeader_1x03_P2.54mm_Vertical
- removed J12: CH3_IN, Connector_PinHeader_2.54mm:PinHeader_1x03_P2.54mm_Vertical
- removed J13: CH4_IN, Connector_PinHeader_2.54mm:PinHeader_1x03_P2.54mm_Vertical
- removed J14: CH1_OUT, Connector_PinHeader_2.54mm:PinHeader_1x03_P2.54mm_Vertical
- removed J15: CH2_OUT, Connector_PinHeader_2.54mm:PinHeader_1x03_P2.54mm_Vertical
- removed J16: CH3_OUT, Connector_PinHeader_2.54mm:PinHeader_1x03_P2.54mm_Vertical
- removed JP2: CH1_MOTOR, Connector_PinHeader_2.54mm:PinHeader_1x03_P2.54mm_Vertical
- removed JP3: CH2, Connector_PinHeader_2.54mm:PinHeader_1x03_P2.54mm_Vertical
- removed JP4: CH3, Connector_PinHeader_2.54mm:PinHeader_1x03_P2.54mm_Vertical
- removed JP5: CH4, Connector_PinHeader_2.54mm:PinHeader_1x03_P2.54mm_Vertical
- removed U1: DS18B20, Package_TO_SOT_THT:TO-92_Inline
- removed kibuzzard-63EE9442: G***, kibuzzard-63EE9442
- removed the kibuzzard-63EE9448 at (168.1, 47.0)
- added C1: 47uF, Capacitor_SMD:C_1206_3216Metric_Pad1.33x1.80mm_HandSolder, F.Cu at (127.2, 37.6)
- added C2: 100nF, Capacitor_SMD:C_1206_3216Metric_Pad1.33x1.80mm_HandSolder, F.Cu at (127.2, 47.5)
- added C3: 47uF, Capacitor_SMD:C_1206_3216Metric_Pad1.33x1.80mm_HandSolder, F.Cu at (127.4, 78.4)
- added C4: 100nF, Capacitor_SMD:C_1206_3216Metric_Pad1.33x1.80mm_HandSolder, F.Cu at (127.2, 52.6)
- added J18: CH1_OUT, Connector_PinHeader_2.54mm:PinHeader_1x03_P2.54mm_Vertical, F.Cu at (172.5, 39.4)
- added J19: CH3_IN, Connector_PinHeader_2.54mm:PinHeader_1x03_P2.54mm_Vertical, F.Cu at (172.5, 61.5)
- added J20: CH3_OUT, Connector_PinHeader_2.54mm:PinHeader_1x03_P2.54mm_Vertical, F.Cu at (172.5, 44.5)
- added J21: CH2_IN, Connector_PinHeader_2.54mm:PinHeader_1x03_P2.54mm_Vertical, F.Cu at (172.5, 64.0)
- added J22: CH2_OUT, Connector_PinHeader_2.54mm:PinHeader_1x03_P2.54mm_Vertical, F.Cu at (172.5, 41.9)
- added J23: CH4_IN, Connector_PinHeader_2.54mm:PinHeader_1x03_P2.54mm_Vertical, F.Cu at (172.5, 58.9)
- added J24: CH4_OUT, Connector_PinHeader_2.54mm:PinHeader_1x03_P2.54mm_Vertical, F.Cu at (172.5, 47.0)
- added JP10: CH2_SERVO, Connector_PinHeader_2.54mm:PinHeader_1x03_P2.54mm_Vertical, F.Cu at (164.4, 49.8)
- added JP11: CH4_SERVO, Connector_PinHeader_2.54mm:PinHeader_1x03_P2.54mm_Vertical, F.Cu at (169.5, 49.8)
- added JP8: CH1_SERVO, Connector_PinHeader_2.54mm:PinHeader_1x03_P2.54mm_Vertical, F.Cu at (161.8, 49.8)
- added JP9: CH3_SERVO, Connector_PinHeader_2.54mm:PinHeader_1x03_P2.54mm_Vertical, F.Cu at (167.0, 49.8)
- added Q3: IRLM2502, Package_TO_SOT_SMD:SOT-23, F.Cu at (158.4, 80.8)
- added Q4: IRLM2502, Package_TO_SOT_SMD:SOT-23, B.Cu at (156.4, 50.9)
- added Q5: IRLM2502, Package_TO_SOT_SMD:SOT-23, B.Cu at (156.4, 54.6)
- added Q6: IRLM2502, Package_TO_SOT_SMD:SOT-23, B.Cu at (156.4, 47.3)
- added R21: 1k, Resistor_SMD:R_1206_3216Metric_Pad1.30x1.75mm_HandSolder, F.Cu at (111.9, 59.3)
- added R22: 1k, Resistor_SMD:R_1206_3216Metric_Pad1.30x1.75mm_HandSolder, F.Cu at (117.2, 59.3)
- added R23: 100, Resistor_SMD:R_1206_3216Metric_Pad1.30x1.75mm_HandSolder, F.Cu at (153.2, 56.0)
- added R24: 1K, Resistor_SMD:R_1206_3216Metric_Pad1.30x1.75mm_HandSolder, F.Cu at (161.8, 45.1)
- added R25: 100, Resistor_SMD:R_1206_3216Metric_Pad1.30x1.75mm_HandSolder, F.Cu at (153.2, 51.0)
- added R26: 1K, Resistor_SMD:R_1206_3216Metric_Pad1.30x1.75mm_HandSolder, F.Cu at (167.0, 45.1)
- added R27: 100, Resistor_SMD:R_1206_3216Metric_Pad1.30x1.75mm_HandSolder, F.Cu at (153.2, 53.5)
- added R28: 1K, Resistor_SMD:R_1206_3216Metric_Pad1.30x1.75mm_HandSolder, F.Cu at (164.5, 45.1)
- added R29: 100, Resistor_SMD:R_1206_3216Metric_Pad1.30x1.75mm_HandSolder, F.Cu at (153.2, 48.6)
- added R30: 1K, Resistor_SMD:R_1206_3216Metric_Pad1.30x1.75mm_HandSolder, F.Cu at (169.5, 45.1)
- added kibuzzard-63F12026: G***, kibuzzard-63F12026, F.Cu at (113.2, 73.1)
- D1: value LED_1 -> LED_R
- D2: value LED_2 -> LED_G
- J17: value CH4_OUT -> CH1_IN
- J3: value BatteryPack -> BATTERY; footprint Connector_PinHeader_2.54mm:PinHeader_1x02_P2.54mm_Vertical -> Connector_PinHeader_2.54mm:PinHeader_1x03_P2.54mm_Vertical
- Q1: value IRLML2502 -> IRLM2502; footprint Package_TO_SOT_SMD:SOT-23_Handsoldering -> Package_TO_SOT_SMD:SOT-23
- Q2: value IRLML2502 -> IRLM2502; footprint Package_TO_SOT_SMD:SOT-23_Handsoldering -> Package_TO_SOT_SMD:SOT-23; moved to B.Cu
- R1: value 300 -> 680
- R10, R11, R12, R20, R8, R9: value 47k -> 10k
- R2: value 300 -> 2k2
- moved J17 19.6 mm to (172.5, 66.5)
- moved Q2 18.5 mm to (156.4, 58.3), turned to 0 degrees
- moved Q1 7.31 mm to (164.0, 75.3), turned to -43.3 degrees
- moved kibuzzard-63F12006 5.47 mm to (114.9, 74.7), turned to 43.699 degrees
- moved J3 4.93 mm to (110.5, 75.6)
- moved R5 2.74 mm to (112.0, 64.0)
- moved R4 2.74 mm to (115.3, 65.5)
- moved R7 1.15 mm to (127.2, 42.5)
- moved kibuzzard-63EE940D 0.54 mm to (168.2, 38.8)
- moved kibuzzard-63EE93FE 0.54 mm to (168.2, 41.4)
Connections:
- J17 pad 2: ESC_5V -> +BATT
- J3 pad 2: Net-(J3-Pin_2) -> +BATT
- Q1 pad 1: LED_2 -> LED_1
- Q1 pad 2: Net-(D1-K) -> MOTOR_SUPPLY_N
- Q1 pad 3: MOTOR_SUPPLY_N -> Net-(D2-K)
- Q2 pad 1: LED_1 -> Net-(Q2-G)
- Q2 pad 2: Net-(D2-K) -> MOTOR_SUPPLY_N
- Q2 pad 3: MOTOR_SUPPLY_N -> Net-(JP8-A)
- R1 pad 1: ESC_5V -> +BATT
- R2 pad 1: ESC_5V -> +BATT
- R7 pad 1: MOTOR_SUPPLY_N -> Net-(U4-EN/CHIP_PU)
- U3 pad 3: Net-(J3-Pin_2) -> +BATT
- U4 pad 10: RUDDER_ADC -> unconnected-(U4-DAC_1/ADC2_CH8/GPIO25-Pad10)
- U4 pad 11: THROTTLE_ADC -> unconnected-(U4-DAC_2/ADC2_CH9/GPIO26-Pad11)
- U4 pad 3: MOTOR_SUPPLY_N -> Net-(U4-EN/CHIP_PU)
- U4 pad 6: unconnected-(U4-GPIO34/ADC1_CH6-Pad6) -> RUDDER_ADC
- U4 pad 7: unconnected-(U4-GPIO35/ADC1_CH7-Pad7) -> THROTTLE_ADC
- U4 pad 8: TEMP_SENSOR -> BATT_SENSOR
Routing:
- net +BATT: track 0.00 -> 153.4 mm, vias 0 -> 1
- net ESC_5V: track 71.7 -> 12.8 mm
- net TEMP_SENSOR: track 35.8 -> 0.00 mm, vias 1 -> 0
- net BATT_SENSOR: track 0.00 -> 27.7 mm, vias 0 -> 2
- net Net-(J14-Pin_1): track 25.8 -> 0.00 mm
- net Net-(J10-Pin_1): track 22.8 -> 0.00 mm
- net Net-(J15-Pin_1): track 20.9 -> 0.00 mm
- net Net-(JP11-A): track 0.00 -> 18.4 mm, vias 0 -> 1
- net Net-(J11-Pin_1): track 18.0 -> 0.00 mm
- net Net-(J18-Pin_1): track 0.00 -> 17.3 mm
- net MOTOR_SUPPLY_N: track 138.7 -> 121.7 mm, vias 8 -> 16
- net Net-(JP9-A): track 0.00 -> 17.0 mm, vias 0 -> 1
- net Net-(J16-Pin_1): track 15.9 -> 0.00 mm
- net CH4_ESP: track 18.2 -> 3.58 mm
- net MOTOR_VOLTAGE: track 48.1 -> 62.7 mm, vias 2 -> 3
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Other:
- board text added: "Gracias a: @spuertes @carlosbetdev @araba_st @kukudrulu @fateuki1 @andygm_ @un_bizco @jfelipe_mg @paco_ggg @vitorio08"
- board text added: "Solar Scavenger v1.1 @LabGluon @Prediktor"
- board text removed: "Gracias a: @spuertes @carlosbetdev @araba_st @kukudrulu @fateuki1 @andygm_ @un_bizco"
- board text removed: "Solar Scavenger v1.0 @LabGluon @Prediktor"
